File: board/psx mister.kicad_pcb (KiCad board)
At the start: 2 copper layers, 85.5 x 25 mm, 13 parts, among them J1 AFB10-S10LCA-00, J2 USB-B-TH_9P-L18.5-W12.0, J3 AV-5, U1 XC6206PxxxMR

Commit message: fixed error
Parts:
- C1, C2: value 1uf -> C_0805
- J1: value AFB10-S10LCA-00 -> Conn_02x05_Odd_Even
- J2: value USB-B-TH_9P-L18.5-W12.0 -> USB3_B
- J3: value AV-5 -> RCJ-044
- R1, R2, R3, R4, R5, R6, R7: value 1K -> R
Connections:
- J2 pad 10: (no net) -> unconnected-(J2-SHIELD-Pad10)
- J2 pad 5: Net-(J1-CMD) -> Net-(J1-CLK)
- J2 pad 6: Net-(J1-IRQ10) -> Net-(J1-DAT)
- J2 pad 8: Net-(J1-CLK) -> Net-(J1-CMD)
- J2 pad 9: Net-(J1-DAT) -> Net-(J1-IRQ10)
Routing:
- net Net-(J1-CLK): track 68.0 -> 75.7 mm, vias 4 -> 5
- net Net-(J1-DAT): track 73.4 -> 80.3 mm, vias 0 -> 1
- net Net-(J1-CMD): track 75.8 -> 69.6 mm
- net Net-(J1-IRQ10): track 84.1 -> 88.6 mm, vias 6 -> 8
- net GND: vias 19 -> 16
