File: board/psx mister.kicad_sch (KiCad schematic)
At the start: 13 parts, among them J1 Conn_02x05_Odd_Even, J2 USB3_B, J3 RCJ-044, U1 XC6206PxxxMR

Commit message: fixed error
Connections:
- net at J1.6 (DAT), R7.2: now also J2.6 (SSTX+); no longer J2.9 (SSRX+)
- net at J1.1 (IRQ10), J3.2, R2.2: now also J2.9 (SSRX+); no longer J2.6 (SSTX+)
- net at J1.10 (CLK), R3.2: now also J2.5 (SSTX-); no longer J2.8 (SSRX-)
- net at J1.8 (CMD), R6.2: now also J2.8 (SSRX-); no longer J2.5 (SSTX-)
Changed lines of the file:
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@@
+	(wire
+		(pts
+			(xy 200.66 97.79) (xy 200.66 109.22)
+		)
+		(stroke
+			(width 0)
+			(type default)
+		)
+	)
+	(wire
+		(pts
+			(xy 203.2 90.17) (xy 203.2 148.59)
+		)
+		(stroke
+			(width 0)
+			(type default)
+		)
+	)
 	(wire
 		(pts
@@
 	(wire
 		(pts
-			(xy 193.04 146.05) (xy 193.04 87.63)
+			(xy 193.04 146.05) (xy 193.04 95.25)
 		)
 		(stroke
@@
 	(wire
 		(pts
+			(xy 203.2 90.17) (xy 187.96 90.17)
+		)
+		(stroke
+			(width 0)
+			(type default)
+		)
+	)
+	(wire
+		(pts
 			(xy 60.96 130.81) (xy 60.96 146.05)
 		)
@@
 	(wire
 		(pts
+			(xy 190.5 87.63) (xy 187.96 87.63)
+		)
+		(stroke
+			(width 0)
+			(type default)
+		)
+	)
+	(wire
+		(pts
 			(xy 134.62 146.05) (xy 134.62 132.08)
 		)
@@
 	(wire
 		(pts
+			(xy 200.66 97.79) (xy 187.96 97.79)
+		)
+		(stroke
+			(width 0)
+			(type default)
+		)
+	)
+	(wire
+		(pts
 			(xy 198.12 143.51) (xy 198.12 82.55)
 		)
@@
 	(wire
 		(pts
-			(xy 190.5 138.43) (xy 190.5 95.25)
+			(xy 190.5 87.63) (xy 190.5 138.43)
 		)
 		(stroke
@@
 	(wire
 		(pts
-			(xy 138.43 148.59) (xy 187.96 148.59)
+			(xy 138.43 148.59) (xy 203.2 148.59)
 		)
 		(stroke
@@
 	(wire
 		(pts
-			(xy 193.04 87.63) (xy 187.96 87.63)
-		)
-		(stroke
-			(width 0)
-			(type default)
-		)
-	)
-	(wire
-		(pts
 			(xy 121.92 81.28) (xy 125.73 81.28)
 		)
@@
 	(wire
 		(pts
-			(xy 187.96 148.59) (xy 187.96 97.79)
+			(xy 187.96 95.25) (xy 193.04 95.25)
 		)
 		(stroke
@@
 	(wire
 		(pts
-			(xy 200.66 90.17) (xy 187.96 90.17)
-		)
-		(stroke
-			(width 0)
-			(type default)
-		)
-	)
-	(wire
-		(pts
 			(xy 146.05 129.54) (xy 146.05 132.08)
 		)
@@
 	(wire
 		(pts
-			(xy 187.96 95.25) (xy 190.5 95.25)
-		)
-		(stroke
-			(width 0)
-			(type default)
-		)
-	)
-	(wire
-		(pts
 			(xy 129.54 106.68) (xy 129.54 119.38)
 		)
 		(stroke
-			(width 0)
-			(type default)
-		)
-	)
-	(wire
-		(pts
-			(xy 200.66 109.22) (xy 200.66 90.17)
-		)
-		(stroke
